Commit message: kbot_mk1

File: src/kbot/description/lidar.xacro (robot description, xacro)
@@ -29,33 +29,3 @@
         </xacro:inertial_cylinder>
     </link>
-<!--
-    <gazebo reference="laser_frame">
-        <material>Gazebo/Black</material>
-        <sensor name="laser" type="ray">
-            <pose> 0 0 0 0 0 0 </pose>
-            <visualize>false</visualize>
-            <update_rate>10</update_rate>
-            <ray>
-                <scan>
-                    <horizontal>
-                        <samples>360</samples>
-                        <min_angle>-3.14</min_angle>
-                        <max_angle>3.14</max_angle>
-                    </horizontal>
-                </scan>
-                <range>
-                    <min>0.3</min>
-                    <max>12</max>
-                </range>
-            </ray>
-            <plugin name="laser_controller" filename="libgazebo_ros_ray_sensor.so">
-                <ros>
-                    <argument>~/out:=scan</argument>
-                </ros>
-                <output_type>sensor_msgs/LaserScan</output_type>
-                <frame_name>laser_frame</frame_name>
-            </plugin>
-        </sensor>
-    </gazebo>
-    -->
 </robot>

Commit message: main

File: src/kbot/description/lidar.xacro (robot description, xacro)
@@ -4,5 +4,5 @@
         <parent link="chassis"/>
         <child  link="laser_frame"/>
-        <origin xyz="0.05 -0.04 0.08" rpy="0 0 0"/>
+        <origin xyz="0.05 -0.05 0.08" rpy="0 0 0"/>
     </joint>
     <link name="laser_frame">

Commit message: kbot_mk1

File: src/kbot/description/lidar.xacro (robot description, xacro)
@@ -4,5 +4,5 @@
         <parent link="chassis"/>
         <child  link="laser_frame"/>
-        <origin xyz="0.05 -0.05 0.08" rpy="0 0 0"/>
+        <origin xyz="0.0 0.0 0.08" rpy="0 0 0"/>           <!-- <origin xyz="0.05 -0.05 0.08" rpy="0 0 0"/> -->
     </joint>
     <link name="laser_frame">
@@ -14,5 +14,5 @@
         </visual>
         <visual>
-            <origin xyz="0 0 -0.05"/>
+            <origin xyz="0.05 -0.05 0.08" rpy="0 0 0"/>       <!-- <origin xyz="0 0 -0.05"/> -->
             <geometry>
                 <cylinder radius="0.01" length="0.1"/>

Commit message: kbot_mk1

File: src/kbot/description/lidar.xacro (robot description, xacro)
@@ -4,8 +4,9 @@
         <parent link="chassis"/>
         <child  link="laser_frame"/>
-        <origin xyz="0.0 0.0 0.08" rpy="0 0 0"/>           <!-- <origin xyz="0.05 -0.05 0.08" rpy="0 0 0"/> -->
+        <origin xyz="0.0 0.0 0.08" rpy="0 0 0"/>             <!-- <origin xyz="0.05 -0.05 0.08" rpy="0 0 0"/> -->
     </joint>
     <link name="laser_frame">
         <visual>
+            <origin xyz="0.05 -0.05 0.00" rpy="0 0 0"/>
             <geometry>
                 <cylinder radius="0.05" length="0.04"/>
@@ -14,5 +15,5 @@
         </visual>
         <visual>
-            <origin xyz="0.05 -0.05 0.08" rpy="0 0 0"/>       <!-- <origin xyz="0 0 -0.05"/> -->
+            <origin xyz="0.05 -0.05 0.00" rpy="0 0 0"/>      <!-- <origin xyz="0 0 -0.05"/> -->
             <geometry>
                 <cylinder radius="0.01" length="0.1"/>
@@ -21,4 +22,5 @@
         </visual>
         <collision>
+            <origin xyz="0.05 -0.05 0.00" rpy="0 0 0"/>
             <geometry>
                 <cylinder radius="0.05" length="0.04"/>
@@ -26,5 +28,5 @@
         </collision>
         <xacro:inertial_cylinder mass="0.1" length="0.04" radius="0.05">
-            <origin xyz="0 0 0" rpy="0 0 0"/>
+            <origin xyz="0.05 -0.05 0.00" rpy="0 0 0"/>      <!-- <origin xyz="0 0 0" rpy="0 0 0"/> -->
         </xacro:inertial_cylinder>
     </link>
